File: EEE3088F Project PCB/EEE3088F Project PCB.kicad_pcb (KiCad board)
At the start: 2 copper layers, 0 parts

Commit message: added a calaculations section, and my motor driver circuit
Parts:
- added J1: JST PH 2.00mm connector, Connector_JST:JST_PH_S2B-PH-K_1x02_P2.00mm_Horizontal, F.Cu at (102.5, 83.0)
- added U1: DRV8833PWP, Package_SO:HTSSOP-16-1EP_4.4x5mm_P0.65mm_EP3.4x5mm_Mask2.46x2.31mm_ThermalVias, F.Cu at (102.2, 61.0)
- added U2: DRV8833PWP, Package_SO:HTSSOP-16-1EP_4.4x5mm_P0.65mm_EP3.4x5mm_Mask2.46x2.31mm_ThermalVias, F.Cu at (103.4, 69.2)
- added am1: 2x16 (2.54mm pin pitch) pin header, Connector_PinHeader_2.54mm:PinHeader_2x16_P2.54mm_Vertical, F.Cu at (89.5, 60.3)
