File: EEE3088F Project PCB/_autosave-EEE3088F Project PCB.kicad_sch (KiCad schematic)
At the start: 15 parts, among them J1 JST PH 2.00mm connector, U1 DRV8833PWR, U2 DRV8833PWPR, U3 INA219AxD

Commit message: added footprints to all motor driver components
Parts:
- C3: footprint (none) -> exported_footprints:CAPC1608X90N
- C5: footprint (none) -> exported_footprints:CAPC1005X55N
- U1, U2: footprint Package_SO:HTSSOP-16-1EP_4.4x5mm_P0.65mm_EP3.4x5mm_Mask2.46x2.31mm_ThermalVias -> exported_footprints:SOP65P640X120-16N
Changed lines of the file:
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@@
+		(polyline
+			(pts
+				(xy 228.6 78.74) (xy 228.6 127) (xy 284.48 127) (xy 284.48 81.28) (xy 281.94 78.74)
+			)
+			(stroke
+				(width 0)
+				(type dash)
+			)
+			(fill
+				(type none)
+			)
+		)
+	)
+	(rule_area
+		(polyline
+			(pts
+				(xy 176.53 165.1) (xy 176.53 127) (xy 285.75 127) (xy 285.75 165.1) (xy 284.48 166.37) (xy 177.8 166.37)
+			)
+			(stroke
+				(width 0)
+				(type dash)
+			)
+			(fill
+				(type none)
+			)
+		)
+	)
+	(rule_area
 		(polyline
 			(pts
@@
 		)
 	)
-	(rule_area
-		(polyline
-			(pts
-				(xy 176.53 165.1) (xy 176.53 127) (xy 285.75 127) (xy 285.75 165.1) (xy 284.48 166.37) (xy 177.8 166.37)
-			)
-			(stroke
-				(width 0)
-				(type dash)
-			)
-			(fill
-				(type none)
-			)
-		)
-	)
-	(rule_area
-		(polyline
-			(pts
-				(xy 228.6 78.74) (xy 228.6 127) (xy 284.48 127) (xy 284.48 81.28) (xy 281.94 78.74)
-			)
-			(stroke
-				(width 0)
-				(type dash)
-			)
-			(fill
-				(type none)
-			)
-		)
-	)
 	(symbol
 		(lib_id "Device:C")
@@
 			)
 		)
-		(property "Footprint" "Package_SO:HTSSOP-16-1EP_4.4x5mm_P0.65mm_EP3.4x5mm_Mask2.46x2.31mm_ThermalVias"
+		(property "Footprint" "exported_footprints:SOP65P640X120-16N"
 			(at 194.31 64.77 0)
 			(effects
@@
 			)
 		)
-		(property "Footprint" ""
+		(property "Footprint" "exported_footprints:CAPC1608X90N"
 			(at 140.0048 25.4 0)
 			(effects
@@
 			)
 		)
-		(property "Footprint" "Package_SO:HTSSOP-16-1EP_4.4x5mm_P0.65mm_EP3.4x5mm_Mask2.46x2.31mm_ThermalVias"
+		(property "Footprint" "exported_footprints:SOP65P640X120-16N"
 			(at 133.35 64.77 0)
 			(effects
@@
 			)
 		)
-		(property "Footprint" ""
+		(property "Footprint" "exported_footprints:CAPC1005X55N"
 			(at 200.9648 25.4 0)
 			(effects
